Commit message: fixpaths

File: src/robot_description/urdf/Pablo_El_Robot.urdf (robot description, URDF)
Before this commit: robot meshesotravez, 5 links, 4 joints
Links:
- link base_castor_link: geometry collision mesh filename=package://robot_description/meshes/base_castor_link.STL; visual mesh filename=package://robot_description/meshes/base_castor_link.STL
- link base_link: geometry collision mesh filename=package://robot_description/meshes/base_link.STL; visual mesh filename=package://robot_description/meshes/base_link.STL
- link wheel_castor_link: geometry collision mesh filename=package://robot_description/meshes/wheel_castor_link.STL; visual mesh filename=package://robot_description/meshes/wheel_castor_link.STL
- link wheel_left_link: geometry collision mesh filename=package://robot_description/meshes/wheel_left_link.STL; visual mesh filename=package://robot_description/meshes/wheel_left_link.STL
- link wheel_right_link: geometry collision mesh filename=package://robot_description/meshes/wheel_right_link.STL; visual mesh filename=package://robot_description/meshes/wheel_right_link.STL
