Commit message: arreglillos namas

File: src/robot_description/urdf/Pablo.urdf.xacro (robot description, xacro)
@@ -12,5 +12,5 @@
       <origin rpy="0 0 0" xyz="-0.002876 -0.00013597 -0.085753"/>
       <mass value="2.4215"/>
-      <inertia ixx="0.0001" ixy="0" ixz="0" iyy="0.0003" iyz="0" izz="0.0002"/>
+      <inertia ixx="0.021858680" ixy="0.0" ixz="0.010020353" iyy="0.078572349" iyz="-0.0" izz="0.091971324"/>
     </inertial>
     <visual>
@@ -19,6 +19,6 @@
         <mesh filename="package://robot_description/meshes/base_link.STL"/>
       </geometry>
-      <material name="ABS">
-        <color rgba="0.79216 0.81961 0.93333 1"/>
+      <material name="naranjitabrillante">
+        <color rgba="1 0.5 0 1"/>
       </material>
     </visual>
@@ -42,5 +42,5 @@
       <origin rpy="0 0 0" xyz="1.3352E-09 8.1843E-10 0.020002"/>
       <mass value="0.26047"/>
-      <inertia ixx="0.00002" ixy="0" ixz="0" iyy="0.00002" iyz="0" izz="0.0001"/>
+      <inertia ixx="0.00008929863" ixy="0" ixz="0" iyy="0.000168983" iyz="0" izz="0.00008929863"/>
     </inertial>
     <visual>
@@ -49,6 +49,6 @@
         <mesh filename="package://robot_description/meshes/wheel_left_link.STL"/>
       </geometry>
-      <material name="NEGRIN">
-        <color rgba="0.90196 0.92157 0.92157 1"/>
+      <material name="negro">
+        <color rgba="0 0 0 1"/>
       </material>
     </visual>
@@ -65,6 +65,6 @@
     <child link="wheel_left_link"/>
     <axis xyz="0 0 1"/>
-    <limit effort="100" velocity="100"/>
-    <dynamics damping="0.1" friction="0.1"/>
+    <limit effort="200" velocity="200"/>
+    <dynamics damping="0.001" friction="0.00001"/>
   </joint>
   <link name="wheel_right_link">
@@ -72,5 +72,5 @@
       <origin rpy="0 0 0" xyz="-1.2885E-09 8.9862E-10 -0.020002"/>
       <mass value="0.26047"/>
-      <inertia ixx="0.00002" ixy="0" ixz="0" iyy="0.00002" iyz="0" izz="0.0001"/>
+      <inertia ixx="0.00008929863" ixy="0" ixz="0" iyy="0.000168983" iyz="0" izz="0.00008929863"/>
     </inertial>
     <visual>
@@ -79,6 +79,6 @@
         <mesh filename="package://robot_description/meshes/wheel_right_link.STL"/>
       </geometry>
-      <material name="">
-        <color rgba="0.90196 0.92157 0.92157 1"/>
+      <material name="negro">
+        <color rgba="0 0 0 1"/>
       </material>
     </visual>
@@ -95,6 +95,6 @@
     <child link="wheel_right_link"/>
     <axis xyz="0 0 1"/>
-    <limit effort="100" velocity="100"/>
-    <dynamics damping="0.1" friction="0.1"/>
+    <limit effort="200" velocity="200"/>
+    <dynamics damping="0.001" friction="0.00001"/>
   </joint>
   <link name="base_castor_link">
@@ -102,5 +102,5 @@
       <origin rpy="0 0 0" xyz="0 -2.08166817117217E-16 0.0141762813814508"/>
       <mass value="0.0128281265837759"/>
-      <inertia ixx="0.00004" ixy="0" ixz="0" iyy="0.00004" iyz="0" izz="0.00001"/>
+      <inertia ixx="0.000008221" ixy="0" ixz="0" iyy="0.000013003" iyz="0" izz="0.000008221"/>
     </inertial>
     <visual>
@@ -109,6 +109,6 @@
         <mesh filename="package://robot_description/meshes/base_castor_link.STL"/>
       </geometry>
-      <material name="OTRO">
-        <color rgba="0.792156862745098 0.819607843137255 0.933333333333333 1"/>
+      <material name="rojo">
+        <color rgba="1 0 0 1"/>
       </material>
     </visual>
@@ -125,6 +125,6 @@
     <child link="base_castor_link"/>
     <axis xyz="0 0 1"/>
-    <limit effort="100" velocity="100"/>
-    <dynamics damping="0.1" friction="0.1"/>
+    <limit effort="200" velocity="200"/>
+    <dynamics damping="0.001" friction="0.00001"/>
   </joint>
   <link name="wheel_castor_link">
@@ -132,5 +132,5 @@
       <origin rpy="0 0 0" xyz="5.67686175845239E-11 -2.52227516650549E-10 -2.34009084454558E-05"/>
       <mass value="0.0459793119455567"/>
-      <inertia ixx="0.00004" ixy="0" ixz="0" iyy="0.00004" iyz="0" izz="0.0001"/>
+      <inertia ixx="0.000004" ixy="0" ixz="0" iyy="0.000004" iyz="0" izz="0.00001"/>
     </inertial>
     <visual>
@@ -139,6 +139,6 @@
         <mesh filename="package://robot_description/meshes/wheel_castor_link.STL"/>
       </geometry>
-      <material name="NOSE">
-        <color rgba="0.901960784313726 0.92156862745098 0.92156862745098 1"/>
+      <material name="negro">
+        <color rgba="0 0 0 1"/>
       </material>
     </visual>
@@ -155,6 +155,82 @@
     <child link="wheel_castor_link"/>
     <axis xyz="0 0 1"/>
-    <limit effort="100" velocity="100"/>
-    <dynamics damping="0.1" friction="0.1"/>
-  </joint>
+    <limit effort="200" velocity="200"/>
+    <dynamics damping="0.001" friction="0.00001"/>
+  </joint>
+  <!-- Gazebo Configuration -->
+  <gazebo reference="base_link">
+    <mu1>200</mu1>
+    <mu2>200</mu2>
+    <kp>1000000</kp>
+    <kd>1</kd>
+    <material>Gazebo/Yellow</material>
+  </gazebo>
+  <gazebo reference="wheel_left_link">
+    <mu1>200</mu1>
+    <mu2>200</mu2>
+    <kp>1000000</kp>
+    <kd>1</kd>
+    <material>Gazebo/Yellow</material>
+  </gazebo>
+  <gazebo reference="wheel_right_link">
+    <mu1>200</mu1>
+    <mu2>200</mu2>
+    <kp>1000000</kp>
+    <kd>1</kd>
+    <material>Gazebo/Yellow</material>
+  </gazebo>
+  <gazebo reference="base_castor_link">
+    <mu1>0.1</mu1>
+    <mu2>0.1</mu2>
+    <kp>1000000</kp>
+    <kd>1</kd>
+    <material>Gazebo/Yellow</material>
+  </gazebo>
+  <gazebo reference="wheel_castor_link">
+    <mu1>1</mu1>
+    <mu2>1</mu2>
+    <kp>1000000</kp>
+    <kd>1</kd>
+    <material>Gazebo/Yellow</material>
+  </gazebo>
+  <gazebo>
+    <plugin name="two_wheeled_robot_diff_drive" filename="libgazebo_ros_diff_drive.so">
+      <update_rate>100</update_rate>
+      <!-- wheels -->
+      <left_joint>wheel_left_link</left_joint>
+      <right_joint>wheel_right_link</right_joint>
+      <!-- kinematics -->
+      <wheel_separation>0.294</wheel_separation>
+      <wheel_diameter>0.08</wheel_diameter>
+      <!-- limits -->
+      <max_wheel_torque>20</max_wheel_torque>
+      <max_wheel_acceleration>20.0</max_wheel_acceleration>
+      <!-- Receive velocity commands on this ROS topic -->
+      <command_topic>cmd_vel</command_topic>
+      <!-- output -->
+      <!-- When false, publish no wheel odometry data to a ROS topic -->
+      <publish_odom>true</publish_odom>
+      <!-- When true, publish coordinate transform from odom to base_footprint -->
+      <!-- I usually use the robot_localization package to publish this transform -->
+      <publish_odom_tf>true</publish_odom_tf>
+      <!-- When true, publish coordinate transform from base_link to the wheels -->
+      <!-- The robot_state_publisher package is often used to publish this transform -->
+      <publish_wheel_tf>true</publish_wheel_tf>
+      <odometry_topic>odom</odometry_topic>
+      <odometry_frame>odom_link</odometry_frame>
+      <robot_base_frame>base_link</robot_base_frame>
+      <odometry_source>1</odometry_source>
+      <ros>
+        <remapping>odom:=wheel/odometry</remapping>
+      </ros>
+    </plugin>
+  </gazebo>
+  <gazebo>
+    <plugin name="gazebo_ros_joint_state_publisher"
+        filename="libgazebo_ros_joint_state_publisher.so">
+        <update_rate>100</update_rate>
+        <joint_name>base_castor_joint</joint_name>
+        <joint_name>wheel_castor_joint</joint_name>
+    </plugin>
+  </gazebo>
 </robot>

File: src/robot_description/urdf/Pablo_El_Robot.urdf (robot description, URDF)
Before this commit: robot Pablo, 5 links, 4 joints
Joints:
- joint base_castor_joint: limit effort=100 velocity=100 -> effort=200 velocity=200
- joint wheel_castor_joint: limit effort=100 velocity=100 -> effort=200 velocity=200
- joint wheel_left_joint: limit effort=100 velocity=100 -> effort=200 velocity=200
- joint wheel_right_joint: limit effort=100 velocity=100 -> effort=200 velocity=200

Commit message: Update robot control and description configurations

File: src/robot_description/urdf/Pablo.urdf.xacro (robot description, xacro)
@@ -164,5 +164,5 @@
     <kp>1000000</kp>
     <kd>1</kd>
-    <material>Gazebo/Yellow</material>
+    <material>Gazebo/Gold</material>
   </gazebo>
   <gazebo reference="wheel_left_link">
@@ -171,5 +171,5 @@
     <kp>1000000</kp>
     <kd>1</kd>
-    <material>Gazebo/Yellow</material>
+    <material>Gazebo/Silver</material>
   </gazebo>
   <gazebo reference="wheel_right_link">
@@ -178,5 +178,5 @@
     <kp>1000000</kp>
     <kd>1</kd>
-    <material>Gazebo/Yellow</material>
+    <material>Gazebo/Silver</material>
   </gazebo>
   <gazebo reference="base_castor_link">
@@ -185,5 +185,5 @@
     <kp>1000000</kp>
     <kd>1</kd>
-    <material>Gazebo/Yellow</material>
+    <material>Gazebo/Black</material>
   </gazebo>
   <gazebo reference="wheel_castor_link">
@@ -192,20 +192,21 @@
     <kp>1000000</kp>
     <kd>1</kd>
-    <material>Gazebo/Yellow</material>
+    <material>Gazebo/Red</material>
   </gazebo>
   <gazebo>
     <plugin name="two_wheeled_robot_diff_drive" filename="libgazebo_ros_diff_drive.so">
-      <update_rate>100</update_rate>
+      <updateRate>100</updateRate>
       <!-- wheels -->
-      <left_joint>wheel_left_link</left_joint>
-      <right_joint>wheel_right_link</right_joint>
+      <leftJoint>wheel_left_joint</leftJoint>
+      <rightJoint>wheel_right_joint</rightJoint>
       <!-- kinematics -->
-      <wheel_separation>0.294</wheel_separation>
-      <wheel_diameter>0.08</wheel_diameter>
+      <wheelSeparation>0.294</wheelSeparation>
+      <wheelDiameter>0.08</wheelDiameter>
       <!-- limits -->
-      <max_wheel_torque>20</max_wheel_torque>
-      <max_wheel_acceleration>20.0</max_wheel_acceleration>
+      <wheelTorque>20</wheelTorque>
+      <maxWheelTorque>20</maxWheelTorque>
+      <wheelAcceleration>20.0</wheelAcceleration>
       <!-- Receive velocity commands on this ROS topic -->
-      <command_topic>cmd_vel</command_topic>
+      <commandTopic>cmd_vel</commandTopic>
       <!-- output -->
       <!-- When false, publish no wheel odometry data to a ROS topic -->
@@ -213,12 +214,13 @@
       <!-- When true, publish coordinate transform from odom to base_footprint -->
       <!-- I usually use the robot_localization package to publish this transform -->
-      <publish_odom_tf>true</publish_odom_tf>
+      <publishOdomTF>true</publishOdomTF>
       <!-- When true, publish coordinate transform from base_link to the wheels -->
       <!-- The robot_state_publisher package is often used to publish this transform -->
-      <publish_wheel_tf>true</publish_wheel_tf>
-      <odometry_topic>odom</odometry_topic>
-      <odometry_frame>odom_link</odometry_frame>
-      <robot_base_frame>base_link</robot_base_frame>
-      <odometry_source>1</odometry_source>
+      <publishWheelTF>true</publishWheelTF>
+      <odometryTopic>odom</odometryTopic>
+      <odometryFrame>odom_link</odometryFrame>
+      <robotBaseFrame>base_link</robotBaseFrame>
+      <publishWheelJointState>true</publishWheelJointState>
+      <odometrySource>1</odometrySource>
       <ros>
         <remapping>odom:=wheel/odometry</remapping>
@@ -229,5 +231,5 @@
     <plugin name="gazebo_ros_joint_state_publisher"
         filename="libgazebo_ros_joint_state_publisher.so">
-        <update_rate>100</update_rate>
+        <updateRate>100</updateRate>
         <joint_name>base_castor_joint</joint_name>
         <joint_name>wheel_castor_joint</joint_name>
